File: hex_schmitt_CMOS.brd (EAGLE design)
At the start: 160 x 100 mm, 24 parts, among them IC1 40106N, J1 AUDIO_JACK_3.5MM_PTH

Commit message: v1, single oscillator pcb works
Parts:
- removed C2, C3, C4, C5, C6: (no value), resistor:E1,8-4
- removed R3, R4, R5, R6, R7: 10K, resistor:0204/5
- removed VR2, VR3, VR4, VR5, VR6: 10k, SparkFun-Resistors:POT-PTH-ALPS
- added H1, H2, H3, H4: STAND-OFF, SparkFun-Hardware:STAND-OFF
- C1: value (none) -> 10u; device resistor:E1,8-4 -> cta_library_EAGLE:E2,5-5
- LED1: value (none) -> Red
- R1: value 330 -> 10k; device resistor:0204/5 -> cta_library_EAGLE:0204/5_66PADS
- R2: value 10K -> 330; device resistor:0204/5 -> cta_library_EAGLE:0204/5_66PADS
- S1: value (none) -> switch
- X1: value (none) -> DC
- moved J1 82.3 mm to (46.1, 16.8), turned to 180 degrees
- moved R2 81.8 mm to (22.9, 39.4), turned to 180 degrees
- moved C1 76.0 mm to (32.1, 6.07)
- moved LED1 73.8 mm to (30.5, 39.4)
- moved R1 65.3 mm to (41.9, 25.4)
- moved VR1 52.8 mm to (30.9, 17.2), turned to 270 degrees
- moved IC1 50.9 mm to (27.9, 30.5)
- moved S1 47.4 mm to (12.5, 39.9), turned to 90 degrees
- moved X1 34.0 mm to (0.51, 29.9), turned to 270 degrees
Connections:
- removed net N$10: IC1.8, R5.1, VR4.P$1
- removed net N$11: C5.+, IC1.11, VR5.P$2
- removed net N$12: IC1.10, R6.1, VR5.P$1
- removed net N$13: C6.+, IC1.13, VR6.P$2
- removed net N$14: IC1.12, R7.1, VR6.P$1
- removed net N$3 (its old number): LED1.A, R1.1
- removed net N$4: IC1.2, R2.1, VR1.P$1
- removed net N$6: IC1.4, R3.1, VR2.P$1
- removed net N$7: C3.+, IC1.5, VR3.P$2
- removed net N$8: IC1.6, R4.1, VR3.P$1
- removed net N$9: C4.+, IC1.9, VR4.P$2
- new net N$2: IC1.2, R1.1, VR1.P$1
- net GND: no longer C2.-, C3.-, C4.-, C5.-, C6.-
- net N$5: now also LED1.A, R2.1; no longer C2.+, IC1.3, VR2.P$2
- net OUT: now also R1.2; no longer R2.2, R3.2, R4.2, R5.2, R6.2, R7.2
- net VCC: now also R2.2; no longer R1.2
Routing:
- net N$2: track 0.00 -> 45.3 mm, vias 0 -> 1
- net N$1: track 0.00 -> 29.4 mm
- net VCC: track 0.00 -> 10.4 mm
- net N$3: track 0.00 -> 8.17 mm
- net OUT: track 0.00 -> 5.05 mm
- net N$5: track 0.00 -> 3.81 mm
- added copper zone on layer 16, net GND
Other:
- board size 160 x 100 mm -> 49.5 x 43 mm

Commit message: screw mounts
Parts:
- moved H4 69.2 mm to (46.2, 3.12)
- moved H2 50.3 mm to (46.2, 40.0)
- moved H3 32.6 mm to (3.23, 3.12)
Changed lines of the file:
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@@
 <attribute name="VALUE" x="-4.698" y="37.846" size="0.6096" layer="27" font="vector" ratio="20" align="top-center"/>
 </element>
-<element name="H2" library="SparkFun-Hardware" library_urn="urn:adsk.eagle:library:519" package="STAND-OFF" package3d_urn="urn:adsk.eagle:package:38630/1" value="STAND-OFF" x="-3.5306" y="32.9438" smashed="yes">
-<attribute name="NAME" x="-3.5306" y="34.9758" size="0.6096" layer="25" font="vector" ratio="20" align="bottom-center"/>
-<attribute name="VALUE" x="-3.5306" y="30.9118" size="0.6096" layer="27" font="vector" ratio="20" align="top-center"/>
+<element name="H2" library="SparkFun-Hardware" library_urn="urn:adsk.eagle:library:519" package="STAND-OFF" package3d_urn="urn:adsk.eagle:package:38630/1" value="STAND-OFF" x="46.228" y="39.9796" smashed="yes">
+<attribute name="NAME" x="46.228" y="42.0116" size="0.6096" layer="25" font="vector" ratio="20" align="bottom-center"/>
+<attribute name="VALUE" x="46.228" y="37.9476" size="0.6096" layer="27" font="vector" ratio="20" align="top-center"/>
 </element>
-<element name="H3" library="SparkFun-Hardware" library_urn="urn:adsk.eagle:library:519" package="STAND-OFF" package3d_urn="urn:adsk.eagle:package:38630/1" value="STAND-OFF" x="-9.8806" y="32.9438" smashed="yes">
-<attribute name="NAME" x="-9.8806" y="34.9758" size="0.6096" layer="25" font="vector" ratio="20" align="bottom-center"/>
-<attribute name="VALUE" x="-9.8806" y="30.9118" size="0.6096" layer="27" font="vector" ratio="20" align="top-center"/>
+<element name="H3" library="SparkFun-Hardware" library_urn="urn:adsk.eagle:library:519" package="STAND-OFF" package3d_urn="urn:adsk.eagle:package:38630/1" value="STAND-OFF" x="3.2258" y="3.1242" smashed="yes">
+<attribute name="NAME" x="3.2258" y="5.1562" size="0.6096" layer="25" font="vector" ratio="20" align="bottom-center"/>
+<attribute name="VALUE" x="3.2258" y="1.0922" size="0.6096" layer="27" font="vector" ratio="20" align="top-center"/>
 </element>
-<element name="H4" library="SparkFun-Hardware" library_urn="urn:adsk.eagle:library:519" package="STAND-OFF" package3d_urn="urn:adsk.eagle:package:38630/1" value="STAND-OFF" x="-16.2306" y="32.9438" smashed="yes">
-<attribute name="NAME" x="-16.2306" y="34.9758" size="0.6096" layer="25" font="vector" ratio="20" align="bottom-center"/>
-<attribute name="VALUE" x="-16.2306" y="30.9118" size="0.6096" layer="27" font="vector" ratio="20" align="top-center"/>
+<element name="H4" library="SparkFun-Hardware" library_urn="urn:adsk.eagle:library:519" package="STAND-OFF" package3d_urn="urn:adsk.eagle:package:38630/1" value="STAND-OFF" x="46.228" y="3.1242" smashed="yes">
+<attribute name="NAME" x="46.228" y="5.1562" size="0.6096" layer="25" font="vector" ratio="20" align="bottom-center"/>
+<attribute name="VALUE" x="46.228" y="1.0922" size="0.6096" layer="27" font="vector" ratio="20" align="top-center"/>
 </element>
 <element name="LED1" library="led" library_urn="urn:adsk.eagle:library:259" package="LED5MM" package3d_urn="urn:adsk.eagle:package:15799/2" value="Red" x="30.48" y="39.37" smashed="yes">
